File: Kicad/sub.kicad_sch (KiCad schematic)
At the start: 16 parts

Commit message: subwoofer fix
Connections:
- net GND: now also R61.1, R62.2
Changed lines of the file:
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@@
+	)
+	(junction
+		(at 186.69 88.9)
+		(diameter 0)
+		(color 0 0 0 0)
 	)
 	(junction
@@
 		)
 		(stroke
+			(width 0)
+			(type default)
+		)
+	)
+	(wire
+		(pts
+			(xy 168.91 88.9) (xy 186.69 88.9)
+		)
+		(stroke
