File: Kicad/volume.kicad_sch (KiCad schematic)
At the start: 1 part

Commit message: moved dac to input path and added input multiplexing
Parts:
- removed RV1: 10k log, Library:10k pot, symbol Device:R_Potentiometer_Dual
