File: Kicad/EQ.kicad_sch (KiCad schematic)
At the start: 30 parts, among them U5 OPA1656ID

Commit message: moved dac to input path and added input multiplexing
Parts:
- R10, R11, R12, R13, R14, R15, R16, R17, R18, R19, R20, R21, R22, R9: footprint Capacitor_SMD:C_0805_2012Metric_Pad1.18x1.45mm_HandSolder -> Resistor_SMD:R_0805_2012Metric_Pad1.20x1.40mm_HandSolder
- R23, R24: footprint Capacitor_SMD:C_1206_3216Metric_Pad1.33x1.80mm_HandSolder -> Resistor_SMD:R_1206_3216Metric_Pad1.30x1.75mm_HandSolder
Connections:
- net GND renamed GNDA
- net left-volume renamed left-input
- net right-volume renamed right-input
Other:
- moved on the sheet: U5C
Changed lines of the file:
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@@
 	(wire
 		(pts
-			(xy 46.99 129.54) (xy 46.99 132.08)
+			(xy 44.45 104.14) (xy 44.45 106.68)
 		)
 		(stroke
@@
 	(wire
 		(pts
-			(xy 26.67 129.54) (xy 29.21 129.54)
+			(xy 24.13 104.14) (xy 26.67 104.14)
 		)
 		(stroke
@@
 	(wire
 		(pts
-			(xy 44.45 129.54) (xy 46.99 129.54)
+			(xy 41.91 104.14) (xy 44.45 104.14)
 		)
 		(stroke
@@
 	(wire
 		(pts
-			(xy 26.67 127) (xy 26.67 129.54)
+			(xy 24.13 101.6) (xy 24.13 104.14)
 		)
 		(stroke
@@
 		)
 	)
-	(hierarchical_label "right-volume"
+	(hierarchical_label "right-input"
 		(shape input)
 		(at 44.45 148.59 180)
@@
 		)
 	)
-	(hierarchical_label "left-volume"
+	(hierarchical_label "left-input"
 		(shape input)
 		(at 44.45 62.23 180)
@@
 			)
 		)
-		(property "Footprint" "Capacitor_SMD:C_0805_2012Metric_Pad1.18x1.45mm_HandSolder"
+		(property "Footprint" "Resistor_SMD:R_0805_2012Metric_Pad1.20x1.40mm_HandSolder"
 			(at 96.52 64.008 90)
 			(hide yes)
@@
 			)
 		)
-		(property "Footprint" "Capacitor_SMD:C_0805_2012Metric_Pad1.18x1.45mm_HandSolder"
+		(property "Footprint" "Resistor_SMD:R_0805_2012Metric_Pad1.20x1.40mm_HandSolder"
 			(at 58.42 150.368 90)
 			(hide yes)
@@
 			)
 		)
-		(property "Value" "GND"
+		(property "Value" "GNDA"
 			(at 134.62 87.63 0)
 			(show_name no)
@@
 			)
 		)
-		(property "Footprint" "Capacitor_SMD:C_0805_2012Metric_Pad1.18x1.45mm_HandSolder"
+		(property "Footprint" "Resistor_SMD:R_0805_2012Metric_Pad1.20x1.40mm_HandSolder"
 			(at 96.52 135.128 90)
 			(hide yes)
@@
 			)
 		)
-		(property "Footprint" "Capacitor_SMD:C_0805_2012Metric_Pad1.18x1.45mm_HandSolder"
+		(property "Footprint" "Resistor_SMD:R_0805_2012Metric_Pad1.20x1.40mm_HandSolder"
 			(at 96.52 150.368 90)
 			(hide yes)
@@
 			)
 		)
-		(property "Footprint" "Capacitor_SMD:C_1206_3216Metric_Pad1.33x1.80mm_HandSolder"
+		(property "Footprint" "Resistor_SMD:R_1206_3216Metric_Pad1.30x1.75mm_HandSolder"
 			(at 114.3 164.592 90)
 			(hide yes)
@@
 			)
 		)
-		(property "Value" "GND"
+		(property "Value" "GNDA"
 			(at 114.3 143.51 0)
 			(show_name no)
@@
 			)
 		)
-		(property "Footprint" "Capacitor_SMD:C_0805_2012Metric_Pad1.18x1.45mm_HandSolder"
+		(property "Footprint" "Resistor_SMD:R_0805_2012Metric_Pad1.20x1.40mm_HandSolder"
 			(at 58.42 174.498 90)
 			(hide yes)
@@
 	(symbol
 		(lib_id "power:+24V")
-		(at 26.67 127 0)
+		(at 24.13 101.6 0)
 		(unit 1)
 		(body_style 1)
@@
 		(dnp no)
 		(property "Reference" "#PWR024"
-			(at 26.67 130.81 0)
+			(at 24.13 105.41 0)
 			(hide yes)
 			(show_name no)
@@
 		)
 		(property "Value" "+12V"
-			(at 26.67 122.428 0)
+			(at 24.13 97.028 0)
 			(show_name no)
 			(do_not_autoplace no)
@@
 		)
 		(property "Footprint" ""
-			(at 26.67 127 0)
+			(at 24.13 101.6 0)
 			(hide yes)
 			(show_name no)
@@
 		)
 		(property "Datasheet" ""
-			(at 26.67 127 0)
+			(at 24.13 101.6 0)
 			(hide yes)
 			(show_name no)
@@
 		)
 		(property "Description" "Power symbol creates a global label with name \"+24V\""
-			(at 26.67 127 0)
+			(at 24.13 101.6 0)
 			(hide yes)
 			(show_name no)
@@
 			)
 		)
-		(property "Footprint" "Capacitor_SMD:C_0805_2012Metric_Pad1.18x1.45mm_HandSolder"
+		(property "Footprint" "Resistor_SMD:R_0805_2012Metric_Pad1.20x1.40mm_HandSolder"
 			(at 96.52 88.138 90)
 			(hide yes)
@@
 			)
 		)
-		(property "Footprint" "Capacitor_SMD:C_0805_2012Metric_Pad1.18x1.45mm_HandSolder"
+		(property "Footprint" "Resistor_SMD:R_0805_2012Metric_Pad1.20x1.40mm_HandSolder"
 			(at 58.42 64.008 90)
 			(hide yes)
@@
 	(symbol
 		(lib_id "Amplifier_Operational:OPA1656ID")
-		(at 36.83 127 90)
+		(at 34.29 101.6 90)
 		(unit 3)
 		(body_style 1)
@@
 		(fields_autoplaced yes)
 		(property "Reference" "U5"
-			(at 36.83 124.46 90)
+			(at 34.29 99.06 90)
 			(show_name no)
 			(do_not_autoplace no)
@@
 		)
 		(property "Value" "OPA1656ID"
-			(at 36.83 127 90)
+			(at 34.29 101.6 90)
 			(show_name no)
 			(do_not_autoplace no)
@@
 		)
 		(property "Footprint" "Package_SO:SOIC-8_3.9x4.9mm_P1.27mm"
-			(at 36.83 127 0)
+			(at 34.29 101.6 0)
 			(hide yes)
 			(show_name no)
@@
 		)
 		(property "Datasheet" "https://www.ti.com/lit/ds/symlink/opa1656.pdf"
-			(at 36.83 127 0)
+			(at 34.29 101.6 0)
 			(hide yes)
 			(show_name no)
@@
 		)
 		(property "Description" "Dual Ultra-Low-Noise, Low-Distortion, FET-Input, Burr-Brown Audio Operational Amplifiers, SOIC-8"
-			(at 36.83 127 0)
+			(at 34.29 101.6 0)
 			(hide yes)
 			(show_name no)
@@
 			)
 		)
-		(property "Footprint" "Capacitor_SMD:C_0805_2012Metric_Pad1.18x1.45mm_HandSolder"
+		(property "Footprint" "Resistor_SMD:R_0805_2012Metric_Pad1.20x1.40mm_HandSolder"
 			(at 96.52 127.508 90)
 			(hide yes)
@@
 			)
 		)
-		(property "Value" "GND"
+		(property "Value" "GNDA"
 			(at 134.62 173.99 0)
 			(show_name no)
@@
 			)
 		)
-		(property "Footprint" "Capacitor_SMD:C_0805_2012Metric_Pad1.18x1.45mm_HandSolder"
+		(property "Footprint" "Resistor_SMD:R_0805_2012Metric_Pad1.20x1.40mm_HandSolder"
 			(at 58.42 88.138 90)
 			(hide yes)
@@
 			)
 		)
-		(property "Footprint" "Capacitor_SMD:C_1206_3216Metric_Pad1.33x1.80mm_HandSolder"
+		(property "Footprint" "Resistor_SMD:R_1206_3216Metric_Pad1.30x1.75mm_HandSolder"
 			(at 114.3 78.232 90)
 			(hide yes)
@@
 			)
 		)
-		(property "Footprint" "Capacitor_SMD:C_0805_2012Metric_Pad1.18x1.45mm_HandSolder"
+		(property "Footprint" "Resistor_SMD:R_0805_2012Metric_Pad1.20x1.40mm_HandSolder"
 			(at 58.42 127.508 90)
 			(hide yes)
@@
 			)
 		)
-		(property "Footprint" "Capacitor_SMD:C_0805_2012Metric_Pad1.18x1.45mm_HandSolder"
+		(property "Footprint" "Resistor_SMD:R_0805_2012Metric_Pad1.20x1.40mm_HandSolder"
 			(at 96.52 174.498 90)
 			(hide yes)
@@
 	(symbol
 		(lib_id "power:-12V")
-		(at 46.99 132.08 180)
+		(at 44.45 106.68 180)
 		(unit 1)
 		(body_style 1)
@@
 		(fields_autoplaced yes)
 		(property "Reference" "#PWR020"
-			(at 46.99 128.27 0)
+			(at 44.45 102.87 0)
 			(hide yes)
 			(show_name no)
@@
 		)
 		(property "Value" "-12V"
-			(at 46.99 137.16 0)
+			(at 44.45 111.76 0)
 			(show_name no)
 			(do_not_autoplace no)
@@
 		)
 		(property "Footprint" ""
-			(at 46.99 132.08 0)
+			(at 44.45 106.68 0)
 			(hide yes)
 			(show_name no)
@@
 		)
 		(property "Datasheet" ""
-			(at 46.99 132.08 0)
+			(at 44.45 106.68 0)
 			(hide yes)
 			(show_name no)
@@
 		)
 		(property "Description" "Power symbol creates a global label with name \"-12V\""
-			(at 46.99 132.08 0)
+			(at 44.45 106.68 0)
 			(hide yes)
 			(show_name no)
@@
 			)
 		)
-		(property "Value" "GND"
+		(property "Value" "GNDA"
 			(at 114.3 57.15 0)
 			(show_name no)
@@
 			)
 		)
-		(property "Footprint" "Capacitor_SMD:C_0805_2012Metric_Pad1.18x1.45mm_HandSolder"
+		(property "Footprint" "Resistor_SMD:R_0805_2012Metric_Pad1.20x1.40mm_HandSolder"
 			(at 96.52 48.768 90)
 			(hide yes)
@@
 			)
 		)
-		(property "Footprint" "Capacitor_SMD:C_0805_2012Metric_Pad1.18x1.45mm_HandSolder"
+		(property "Footprint" "Resistor_SMD:R_0805_2012Metric_Pad1.20x1.40mm_HandSolder"
 			(at 96.52 41.148 90)
 			(hide yes)
@@
 			)
 		)
-		(property "Footprint" "Capacitor_SMD:C_0805_2012Metric_Pad1.18x1.45mm_HandSolder"
+		(property "Footprint" "Resistor_SMD:R_0805_2012Metric_Pad1.20x1.40mm_HandSolder"
 			(at 58.42 41.148 90)
 			(hide yes)

Commit message: final schematic
Connections:
- net GNDA renamed GND
Other:
- moved on the sheet: C13, C14, C15, C16, C17, C18, C19, C20, C21, C22, R10, R11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
