File: Kicad/dac.kicad_sch (KiCad schematic)
At the start: 16 parts, among them U14 PCM5102A

Commit message: moved dac to input path and added input multiplexing
Connections:
- net AGND: no longer C47.1, C48.2
- new net GNDA: C47.1, C48.2
Changed lines of the file:
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@@
 			)
 		)
-		(property "Value" "AGND"
+		(property "Value" "GNDA"
 			(at 133.604 85.598 0)
 			(show_name no)
@@
 			)
 		)
-		(property "Value" "AGND"
+		(property "Value" "GNDA"
 			(at 120.904 85.598 0)
 			(show_name no)

Commit message: final schematic
Connections:
- net AGND is gone; now on net GND: C44.1, C46.2, U14.9 (AGND)
- net GNDA is gone; now on net GND: C47.1, C48.2
Changed lines of the file:
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@@
 			)
 		)
-		(property "Value" "GNDA"
+		(property "Value" "GND"
 			(at 133.604 85.598 0)
 			(show_name no)
@@
 		(in_pos_files yes)
 		(dnp no)
-		(fields_autoplaced yes)
 		(property "Reference" "#PWR049"
 			(at 129.54 97.79 0)
@@
 		)
 		(property "Value" "+3.3V"
-			(at 129.54 88.9 0)
+			(at 133.858 91.948 0)
 			(show_name no)
 			(do_not_autoplace no)
@@
 			)
 		)
-		(property "Value" "AGND"
+		(property "Value" "GND"
 			(at 133.604 103.378 0)
 			(show_name no)
@@
 			)
 		)
-		(property "Value" "GNDA"
+		(property "Value" "GND"
 			(at 120.904 85.598 0)
 			(show_name no)
