File: Kicad/amp.kicad_sch (KiCad schematic)
At the start: 41 parts, among them Q1 Q_NMOS_DGS, Q2 Q_NMOS_DGS, U12 TPA3221DDV, U13 TPA3221DDV

Commit message: subwoofer fix
Connections:
- net Stereo Right Channel/OUT_M: now also U12.27 (OUT2_M), U12.28 (OUT2_M__1); no longer U12.32 (OUT2_P)
- net Stereo Right Channel/OUT_P: now also U12.32 (OUT2_P); no longer U12.27 (OUT2_M), U12.28 (OUT2_M__1)
Changed lines of the file:
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@@
 	(wire
 		(pts
-			(xy 196.85 58.42) (xy 180.34 58.42)
-		)
-		(stroke
-			(width 0)
-			(type default)
-		)
-	)
-	(wire
-		(pts
 			(xy 54.61 80.01) (xy 86.36 80.01)
 		)
@@
 	(wire
 		(pts
-			(xy 196.85 63.5) (xy 182.88 63.5)
-		)
-		(stroke
-			(width 0)
-			(type default)
-		)
-	)
-	(wire
-		(pts
 			(xy 121.92 57.15) (xy 124.46 57.15)
 		)
@@
 	(wire
 		(pts
+			(xy 182.88 63.5) (xy 196.85 63.5)
+		)
+		(stroke
+			(width 0)
+			(type default)
+		)
+	)
+	(wire
+		(pts
 			(xy 86.36 72.39) (xy 83.82 72.39)
 		)
@@
 	(wire
 		(pts
+			(xy 180.34 58.42) (xy 196.85 58.42)
+		)
+		(stroke
+			(width 0)
+			(type default)
+		)
+	)
+	(wire
+		(pts
 			(xy 86.36 54.61) (xy 83.82 54.61)
 		)
@@
 		)
 		(pin "OUT_P" input
-			(at 196.85 63.5 180)
+			(at 196.85 58.42 180)
 			(effects
 				(font
@@
 		)
 		(pin "OUT_M" input
-			(at 196.85 58.42 180)
+			(at 196.85 63.5 180)
 			(effects
 				(font

Commit message: moved dac to input path and added input multiplexing
Connections:
- net channel1-in2 is gone; now on net GND: C71.1
- net channel2-in2 is gone; now on net GND: C74.1
- net sub-in2 is gone; now on net GND: C81.1

Commit message: fixed issues in amp
Parts:
- removed R52: 5.6k, Resistor_SMD:R_1206_3216Metric_Pad1.30x1.75mm_HandSolder, symbol Device:R
- added R70, R71: 39k, Resistor_SMD:R_1206_3216Metric_Pad1.30x1.75mm_HandSolder, symbol Device:R
- added R72: 100k, Resistor_SMD:R_1206_3216Metric_Pad1.30x1.75mm_HandSolder, symbol Device:R
- R56: value 5.6k -> 100k
Connections:
- net +5V: now also R70.1, R72.1
- net GND: now also R71.1
- net at R56.2, U13.2 (GAIN/SLV): now also R70.2
- net at U12.2 (GAIN/SLV): now also R71.2, R72.2
Other:
- moved on the sheet: R56, R69
