File: Kicad/esp32.kicad_sch (KiCad schematic)
At the start: 24 parts, among them J2 Display, J4 pad, J5 pad, J6 pad, J7 UART, J8 pad, J9 pad, U11 ESP32-WROOM-32UE-N16, U16 XL1509-3.3

Commit message: subwoofer fix
Parts:
- added J3: LED, symbol Connector:Conn_01x02_Pin
- added R2: 220, symbol Device:R
Connections:
- net GND: now also J3.2 (Pin_2)
- net at U11.11 (IO26): now also R2.2
- new net: J3.1 (Pin_1), R2.1
- no-connect marks 5 -> 4
Other:
- moved on the sheet: J8

Commit message: moved dac to input path and added input multiplexing
Parts:
- removed J4, J5, J6, J8, J9: pad, symbol Connector:Conn_01x01_Pin
- added TP1: io0, symbol Connector:TestPoint
- added TP3: gnd, symbol Connector:TestPoint
- added TP4: 3.3, symbol Connector:TestPoint
- added TP5: en, symbol Connector:TestPoint
- R47, R48, R49, R50, R66, R7: footprint Capacitor_SMD:C_0805_2012Metric_Pad1.18x1.45mm_HandSolder -> Resistor_SMD:R_0805_2012Metric_Pad1.20x1.40mm_HandSolder
Connections:
- net +3.3V: now also TP4.1
- net GND: now also TP3.1
- net SCL: now reaches J2.2 (Pin_2), U11.36 (IO22)
- net SDA: now reaches J2.3 (Pin_3), U11.37 (IO23)
- net at C41.1, R7.2, U11.3 (EN): now also TP5.1
- net at R47.2, U11.25 (IO0): now also TP1.1
- net select: now reaches U11.28 (IO17)
- no-connect marks 4 -> 3
Other:
- added sheet Power measurement (Power measurement.kicad_sch)
- moved on the sheet: R48

Commit message: final schematic
Changed lines of the file:
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@@
 	(wire
 		(pts
-			(xy 82.55 129.54) (xy 85.09 129.54)
+			(xy 67.31 129.54) (xy 69.85 129.54)
 		)
 		(stroke
@@
 	(wire
 		(pts
-			(xy 82.55 121.92) (xy 86.36 121.92)
+			(xy 67.31 121.92) (xy 71.12 121.92)
 		)
 		(stroke
@@
 	(wire
 		(pts
-			(xy 82.55 127) (xy 85.09 127)
+			(xy 67.31 127) (xy 69.85 127)
 		)
 		(stroke
@@
 	(wire
 		(pts
-			(xy 58.42 156.21) (xy 62.23 156.21)
+			(xy 43.18 156.21) (xy 46.99 156.21)
 		)
 		(stroke
@@
 	(wire
 		(pts
-			(xy 92.71 158.75) (xy 88.9 158.75)
+			(xy 77.47 158.75) (xy 73.66 158.75)
 		)
 		(stroke
@@
 	(wire
 		(pts
-			(xy 82.55 116.84) (xy 86.36 116.84)
+			(xy 67.31 116.84) (xy 71.12 116.84)
 		)
 		(stroke
@@
 	(wire
 		(pts
-			(xy 58.42 158.75) (xy 62.23 158.75)
+			(xy 43.18 158.75) (xy 46.99 158.75)
 		)
 		(stroke
@@
 	(wire
 		(pts
-			(xy 82.55 114.3) (xy 86.36 114.3)
+			(xy 67.31 114.3) (xy 71.12 114.3)
 		)
 		(stroke
@@
 	(wire
 		(pts
-			(xy 92.71 156.21) (xy 88.9 156.21)
+			(xy 77.47 156.21) (xy 73.66 156.21)
 		)
 		(stroke
@@
 	(wire
 		(pts
-			(xy 82.55 119.38) (xy 86.36 119.38)
+			(xy 67.31 119.38) (xy 71.12 119.38)
 		)
 		(stroke
@@
 	(global_label "BCK"
 		(shape input)
-		(at 86.36 119.38 0)
+		(at 71.12 119.38 0)
 		(fields_autoplaced yes)
 		(effects
@@
 		)
 		(property "Intersheetrefs" "${INTERSHEET_REFS}"
-			(at 93.1552 119.38 0)
+			(at 77.9152 119.38 0)
 			(hide yes)
 			(show_name no)
@@
 	(global_label "SCL"
 		(shape input)
-		(at 92.71 156.21 0)
+		(at 77.47 156.21 0)
 		(fields_autoplaced yes)
 		(effects
@@
 		)
 		(property "Intersheetrefs" "${INTERSHEET_REFS}"
-			(at 99.2028 156.21 0)
+			(at 83.9628 156.21 0)
 			(hide yes)
 			(show_name no)
@@
 	(global_label "XSMT"
 		(shape input)
-		(at 86.36 121.92 0)
+		(at 71.12 121.92 0)
 		(fields_autoplaced yes)
 		(effects
@@
 		)
 		(property "Intersheetrefs" "${INTERSHEET_REFS}"
-			(at 94.1832 121.92 0)
+			(at 78.9432 121.92 0)
 			(hide yes)
 			(show_name no)
@@
 	(global_label "SDA"
 		(shape input)
-		(at 92.71 158.75 0)
+		(at 77.47 158.75 0)
 		(fields_autoplaced yes)
 		(effects
@@
 		)
 		(property "Intersheetrefs" "${INTERSHEET_REFS}"
-			(at 99.2633 158.75 0)
+			(at 84.0233 158.75 0)
 			(hide yes)
 			(show_name no)
@@
 	(global_label "LRCK"
 		(shape input)
-		(at 86.36 114.3 0)
+		(at 71.12 114.3 0)
 		(fields_autoplaced yes)
 		(effects
@@
 		)
 		(property "Intersheetrefs" "${INTERSHEET_REFS}"
-			(at 94.1833 114.3 0)
+			(at 78.9433 114.3 0)
 			(hide yes)
 			(show_name no)
@@
 	(global_label "DIN"
 		(shape input)
-		(at 86.36 116.84 0)
+		(at 71.12 116.84 0)
 		(fields_autoplaced yes)
 		(effects
@@
 		)
 		(property "Intersheetrefs" "${INTERSHEET_REFS}"
-			(at 92.5505 116.84 0)
+			(at 77.3105 116.84 0)
 			(hide yes)
 			(show_name no)
@@
 	(hierarchical_label "Left Channel"
 		(shape output)
-		(at 85.09 127 0)
+		(at 69.85 127 0)
 		(effects
 			(font
@@
 	(hierarchical_label "Right Channel"
 		(shape output)
-		(at 85.09 129.54 0)
+		(at 69.85 129.54 0)
 		(effects
 			(font
@@
 	(hierarchical_label "In-"
 		(shape input)
-		(at 58.42 158.75 180)
+		(at 43.18 158.75 180)
 		(effects
 			(font
@@
 	(hierarchical_label "In+"
 		(shape input)
-		(at 58.42 156.21 180)
+		(at 43.18 156.21 180)
 		(effects
 			(font
@@
 	)
 	(sheet
-		(at 63.5 111.76)
+		(at 48.26 111.76)
 		(size 19.05 20.32)
 		(exclude_from_sim no)
@@
 		)
 		(property "Sheetname" "DAC"
-			(at 63.5 111.0484 0)
+			(at 48.26 111.0484 0)
 			(show_name no)
 			(do_not_autoplace no)
@@
 		)
 		(property "Sheetfile" "dac.kicad_sch"
-			(at 63.5 132.6646 0)
+			(at 48.26 132.6646 0)
 			(hide yes)
 			(show_name no)
@@
 		)
 		(pin "Right Channel" output
-			(at 82.55 129.54 0)
+			(at 67.31 129.54 0)
 			(effects
 				(font
@@
 		)
 		(pin "Left Channel" output
-			(at 82.55 127 0)
+			(at 67.31 127 0)
 			(effects
 				(font
@@
 		)
 		(pin "LRCK" input
-			(at 82.55 114.3 0)
+			(at 67.31 114.3 0)
 			(effects
 				(font
@@
 		)
 		(pin "BCK" input
-			(at 82.55 119.38 0)
+			(at 67.31 119.38 0)
 			(effects
 				(font
@@
 		)
 		(pin "DIN" input
-			(at 82.55 116.84 0)
+			(at 67.31 116.84 0)
 			(effects
 				(font
@@
 		)
 		(pin "XSMT" input
-			(at 82.55 121.92 0)
+			(at 67.31 121.92 0)
 			(effects
 				(font
@@
 	)
 	(sheet
-		(at 62.23 152.654)
+		(at 46.99 152.654)
 		(size 26.67 8.89)
 		(exclude_from_sim no)
@@
 		)
 		(property "Sheetname" "Power measurement"
-			(at 62.23 151.9424 0)
+			(at 46.99 151.9424 0)
 			(show_name no)
 			(do_not_autoplace no)
@@
 		)
 		(property "Sheetfile" "Power measurement.kicad_sch"
-			(at 62.23 162.1286 0)
+			(at 46.99 162.1286 0)
 			(hide yes)
 			(show_name no)
@@
 		)
 		(pin "SDA" input
-			(at 88.9 158.75 0)
+			(at 73.66 158.75 0)
 			(effects
 				(font
@@
 		)
 		(pin "SCL" input
-			(at 88.9 156.21 0)
+			(at 73.66 156.21 0)
 			(effects
 				(font
@@
 		)
 		(pin "In+" input
-			(at 62.23 156.21 180)
+			(at 46.99 156.21 180)
 			(effects
 				(font
@@
 		)
 		(pin "In-" input
-			(at 62.23 158.75 180)
+			(at 46.99 158.75 180)
 			(effects
 				(font

Commit message: fixed issues in amp
Parts:
- removed R48: 10k, Resistor_SMD:R_0805_2012Metric_Pad1.20x1.40mm_HandSolder, symbol Device:R
Connections:
- no-connect marks 3 -> 4
Changed lines of the file:
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@@
 	)
 	(junction
-		(at 246.38 105.41)
-		(diameter 0)
-		(color 0 0 0 0)
-	)
-	(junction
 		(at 55.88 52.07)
 		(diameter 0)
@@
 	)
 	(no_connect
+		(at 222.25 105.41)
+	)
+	(no_connect
 		(at 222.25 107.95)
 	)
@@
 	(wire
 		(pts
-			(xy 67.31 129.54) (xy 69.85 129.54)
+			(xy 85.09 101.6) (xy 87.63 101.6)
 		)
 		(stroke
@@
 	(wire
 		(pts
-			(xy 67.31 121.92) (xy 71.12 121.92)
+			(xy 85.09 93.98) (xy 88.9 93.98)
 		)
 		(stroke
@@
 	(wire
 		(pts
-			(xy 67.31 127) (xy 69.85 127)
+			(xy 85.09 99.06) (xy 87.63 99.06)
 		)
 		(stroke
@@
 	(wire
 		(pts
-			(xy 43.18 156.21) (xy 46.99 156.21)
+			(xy 72.39 114.3) (xy 76.2 114.3)
 		)
 		(stroke
@@
 	(wire
 		(pts
-			(xy 77.47 158.75) (xy 73.66 158.75)
+			(xy 106.68 116.84) (xy 102.87 116.84)
 		)
 		(stroke
@@
 	(wire
 		(pts
-			(xy 222.25 105.41) (xy 232.41 105.41)
-		)
-		(stroke
-			(width 0)
-			(type default)
-		)
-	)
-	(wire
-		(pts
-			(xy 67.31 116.84) (xy 71.12 116.84)
+			(xy 85.09 88.9) (xy 88.9 88.9)
 		)
 		(stroke
@@
 	(wire
 		(pts
-			(xy 43.18 158.75) (xy 46.99 158.75)
+			(xy 72.39 116.84) (xy 76.2 116.84)
 		)
 		(stroke
@@
 	(wire
 		(pts
-			(xy 240.03 105.41) (xy 246.38 105.41)
-		)
-		(stroke
-			(width 0)
-			(type default)
-		)
-	)
-	(wire
-		(pts
 			(xy 64.77 66.04) (xy 74.93 66.04)
 		)
@@
 	(wire
 		(pts
-			(xy 67.31 114.3) (xy 71.12 114.3)
+			(xy 85.09 86.36) (xy 88.9 86.36)
 		)
 		(stroke
@@
 	(wire
 		(pts
-			(xy 77.47 156.21) (xy 73.66 156.21)
+			(xy 106.68 114.3) (xy 102.87 114.3)
 		)
 		(stroke
@@
 	(wire
 		(pts
-			(xy 67.31 119.38) (xy 71.12 119.38)
+			(xy 85.09 91.44) (xy 88.9 91.44)
 		)
 		(stroke
@@
 	(global_label "BCK"
 		(shape input)
-		(at 71.12 119.38 0)
+		(at 88.9 91.44 0)
 		(fields_autoplaced yes)
 		(effects
@@
 		)
 		(property "Intersheetrefs" "${INTERSHEET_REFS}"
-			(at 77.9152 119.38 0)
+			(at 95.6952 91.44 0)
 			(hide yes)
 			(show_name no)
@@
 	(global_label "SCL"
 		(shape input)
-		(at 77.47 156.21 0)
+		(at 106.68 114.3 0)
 		(fields_autoplaced yes)
 		(effects
@@
 		)
 		(property "Intersheetrefs" "${INTERSHEET_REFS}"
-			(at 83.9628 156.21 0)
+			(at 113.1728 114.3 0)
 			(hide yes)
 			(show_name no)
@@
 	(global_label "XSMT"
 		(shape input)
-		(at 71.12 121.92 0)
+		(at 88.9 93.98 0)
 		(fields_autoplaced yes)
 		(effects
@@
 		)
 		(property "Intersheetrefs" "${INTERSHEET_REFS}"
-			(at 78.9432 121.92 0)
+			(at 96.7232 93.98 0)
 			(hide yes)
 			(show_name no)
@@
 	(global_label "SDA"
 		(shape input)
-		(at 77.47 158.75 0)
+		(at 106.68 116.84 0)
 		(fields_autoplaced yes)
 		(effects
@@
 		)
 		(property "Intersheetrefs" "${INTERSHEET_REFS}"
-			(at 84.0233 158.75 0)
+			(at 113.2333 116.84 0)
 			(hide yes)
 			(show_name no)
@@
 	(global_label "LRCK"
 		(shape input)
-		(at 71.12 114.3 0)
+		(at 88.9 86.36 0)
 		(fields_autoplaced yes)
 		(effects
@@
 		)
 		(property "Intersheetrefs" "${INTERSHEET_REFS}"
-			(at 78.9433 114.3 0)
+			(at 96.7233 86.36 0)
 			(hide yes)
 			(show_name no)
@@
 	(global_label "DIN"
 		(shape input)
-		(at 71.12 116.84 0)
+		(at 88.9 88.9 0)
 		(fields_autoplaced yes)
 		(effects
@@
 		)
 		(property "Intersheetrefs" "${INTERSHEET_REFS}"
-			(at 77.3105 116.84 0)
+			(at 95.0905 88.9 0)
 			(hide yes)
 			(show_name no)
@@
 	(hierarchical_label "Left Channel"
 		(shape output)
-		(at 69.85 127 0)
+		(at 87.63 99.06 0)
 		(effects
 			(font
@@
 	(hierarchical_label "Right Channel"
 		(shape output)
-		(at 69.85 129.54 0)
+		(at 87.63 101.6 0)
 		(effects
 			(font
@@
 	(hierarchical_label "In-"
 		(shape input)
-		(at 43.18 158.75 180)
+		(at 72.39 116.84 180)
 		(effects
 			(font
@@
 	(hierarchical_label "In+"
 		(shape input)
-		(at 43.18 156.21 180)
+		(at 72.39 114.3 180)
 		(effects
 			(font
@@
 	)
 	(symbol
-		(lib_id "Device:R")
-		(at 236.22 105.41 270)
-		(unit 1)
-		(body_style 1)
-		(exclude_from_sim no)
-		(in_bom yes)
-		(on_board yes)
-		(in_pos_files yes)
-		(dnp no)
-		(property "Reference" "R48"
-			(at 234.188 107.696 90)
-			(show_name no)
-			(do_not_autoplace no)
-			(effects
-				(font
-					(size 1.27 1.27)
-				)
-				(justify left)
-			)
-		)
-		(property "Value" "10k"
-			(at 234.188 109.474 90)
-			(show_name no)
-			(do_not_autoplace no)
-			(effects
-				(font
-					(size 1.27 1.27)
-				)
-				(justify left)
-			)
-		)
-		(property "Footprint" "Resistor_SMD:R_0805_2012Metric_Pad1.20x1.40mm_HandSolder"
-			(at 236.22 103.632 90)
-			(hide yes)
-			(show_name no)
-			(do_not_autoplace no)
-			(effects
-				(font
-					(size 1.27 1.27)
-				)
-			)
-		)
-		(property "Datasheet" ""
-			(at 236.22 105.41 0)
-			(hide yes)
-			(show_name no)
-			(do_not_autoplace no)
-			(effects
-				(font
-					(size 1.27 1.27)
-				)
-			)
-		)
-		(property "Description" "Resistor"
-			(at 236.22 105.41 0)
-			(hide yes)
-			(show_name no)
-			(do_not_autoplace no)
-			(effects
-				(font
-					(size 1.27 1.27)
-				)
-			)
-		)
-		(pin "2"
-		)
-		(pin "1"
-		)
-		(instances
-			(project "SoundSystem"
-				(path "/ef5bdc6f-cba8-49ce-9423-d6c9041fdb9d/3e42e31f-f69c-48fe-9507-d66053da3ffa"
-					(reference "R48")
-					(unit 1)
-				)
-			)
-		)
-	)
-	(symbol
 		(lib_id "Connector:Conn_01x04_Pin")
 		(at 270.51 90.17 180)
@@
 	)
 	(sheet
-		(at 48.26 111.76)
+		(at 66.04 83.82)
 		(size 19.05 20.32)
 		(exclude_from_sim no)
@@
 		)
 		(property "Sheetname" "DAC"
-			(at 48.26 111.0484 0)
+			(at 66.04 83.1084 0)
 			(show_name no)
 			(do_not_autoplace no)
@@
 		)
 		(property "Sheetfile" "dac.kicad_sch"
-			(at 48.26 132.6646 0)
+			(at 66.04 104.7246 0)
 			(hide yes)
 			(show_name no)
@@
 		)
 		(pin "Right Channel" output
-			(at 67.31 129.54 0)
+			(at 85.09 101.6 0)
 			(effects
 				(font
@@
 		)
 		(pin "Left Channel" output
-			(at 67.31 127 0)
+			(at 85.09 99.06 0)
 			(effects
 				(font
@@
 		)
 		(pin "LRCK" input
-			(at 67.31 114.3 0)
+			(at 85.09 86.36 0)
 			(effects
 				(font
@@
 		)
 		(pin "BCK" input
-			(at 67.31 119.38 0)
+			(at 85.09 91.44 0)
 			(effects
 				(font
@@
 		)
 		(pin "DIN" input
-			(at 67.31 116.84 0)
+			(at 85.09 88.9 0)
 			(effects
 				(font
@@
 		)
 		(pin "XSMT" input
-			(at 67.31 121.92 0)
+			(at 85.09 93.98 0)
 			(effects
 				(font
@@
 	)
 	(sheet
-		(at 46.99 152.654)
+		(at 76.2 110.744)
 		(size 26.67 8.89)
 		(exclude_from_sim no)
@@
 		)
 		(property "Sheetname" "Power measurement"
-			(at 46.99 151.9424 0)
+			(at 76.2 110.0324 0)
 			(show_name no)
 			(do_not_autoplace no)
@@
 		)
 		(property "Sheetfile" "Power measurement.kicad_sch"
-			(at 46.99 162.1286 0)
+			(at 76.2 120.2186 0)
 			(hide yes)
 			(show_name no)
@@
 		)
 		(pin "SDA" input
-			(at 73.66 158.75 0)
+			(at 102.87 116.84 0)
 			(effects
 				(font
@@
 		)
 		(pin "SCL" input
-			(at 73.66 156.21 0)
+			(at 102.87 114.3 0)
 			(effects
 				(font
@@
 		)
 		(pin "In+" input
-			(at 46.99 156.21 180)
+			(at 76.2 114.3 180)
 			(effects
 				(font
@@
 		)
 		(pin "In-" input
-			(at 46.99 158.75 180)
+			(at 76.2 116.84 180)
 			(effects
 				(font
